File: flexor_wireless/flexor_wireless.kicad_sch (KiCad schematic)
At the start: 0 parts

Commit message: feat: add project metadata to KiCad files
- Add comments, revision, title and issue date to schematic and PCB
- Update project information for flexor_wired variant
- Update project information for flexor_wireless variant
Other:
- title: (none) -> Flexor Keyboard - Wireless
Changed lines of the file:
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@@
 	(generator_version "9.0")
 	(paper "A4")
+	(title_block
+		(title "Flexor Keyboard - Wireless")
+		(date "2025-08-14")
+		(rev "A")
+		(comment 1 "Wireless Version")
+		(comment 2 "34-Key Split Ergonomic Keyboard")
+		(comment 4 "F L E X O R")
+	)
 	(sheet_instances
 		(path "/"
