File: flexor_wired/flexor_wired.kicad_pcb (KiCad board)
At the start: 2 copper layers, 0 parts

Commit message: feat: update PCB design and project configuration
- Update flexor_wired PCB layout and schematic
- Update project configuration and preferences
- Update footprint info cache
Parts:
- added D1: 1N4148W, Diode:1N4148W_SOD-123_SMD, F.Cu at (30.8, 95.3)
- added D10: 1N4148W, Diode:1N4148W_SOD-123_SMD, F.Cu at (111.5, 91.7)
- added D11: 1N4148W, Diode:1N4148W_SOD-123_SMD, F.Cu at (41.3, 127.6)
- added D12: 1N4148W, Diode:1N4148W_SOD-123_SMD, F.Cu at (57.1, 111.7)
- added D13: 1N4148W, Diode:1N4148W_SOD-123_SMD, F.Cu at (74.8, 100.3)
- added D14: 1N4148W, Diode:1N4148W_SOD-123_SMD, F.Cu at (93.5, 113.0)
- added D15: 1N4148W, Diode:1N4148W_SOD-123_SMD, F.Cu at (111.5, 108.7)
- added D16: 1N4148W, Diode:1N4148W_SOD-123_SMD, F.Cu at (110.8, 131.3)
- added D17: 1N4148W, Diode:1N4148W_SOD-123_SMD, F.Cu at (128.6, 134.2)
- added D18: 1N4148W, Diode:1N4148W_SOD-123_SMD, F.Cu at (188.5, 74.7)
- added D19: 1N4148W, Diode:1N4148W_SOD-123_SMD, F.Cu at (206.5, 79.0)
- added D2: 1N4148W, Diode:1N4148W_SOD-123_SMD, F.Cu at (51.7, 78.1)
- added D20: 1N4148W, Diode:1N4148W_SOD-123_SMD, F.Cu at (227.0, 66.4)
- added D21: 1N4148W, Diode:1N4148W_SOD-123_SMD, F.Cu at (248.3, 78.1)
- added D22: 1N4148W, Diode:1N4148W_SOD-123_SMD, F.Cu at (269.2, 95.3)
- added D23: 1N4148W, Diode:1N4148W_SOD-123_SMD, F.Cu at (188.5, 91.7)
- added D24: 1N4148W, Diode:1N4148W_SOD-123_SMD, F.Cu at (206.5, 96.0)
- added D25: 1N4148W, Diode:1N4148W_SOD-123_SMD, F.Cu at (226.1, 83.3)
- added D26: 1N4148W, Diode:1N4148W_SOD-123_SMD, F.Cu at (245.6, 94.9)
- added D27: 1N4148W, Diode:1N4148W_SOD-123_SMD, F.Cu at (264.0, 111.5)
- added D28: 1N4148W, Diode:1N4148W_SOD-123_SMD, F.Cu at (188.5, 108.7)
- added D29: 1N4148W, Diode:1N4148W_SOD-123_SMD, F.Cu at (206.5, 113.0)
- added D3: 1N4148W, Diode:1N4148W_SOD-123_SMD, F.Cu at (73.0, 66.4)
- added D30: 1N4148W, Diode:1N4148W_SOD-123_SMD, F.Cu at (225.2, 100.3)
- added D31: 1N4148W, Diode:1N4148W_SOD-123_SMD, F.Cu at (243.0, 111.7)
- added D32: 1N4148W, Diode:1N4148W_SOD-123_SMD, F.Cu at (258.7, 127.6)
- added D33: 1N4148W, Diode:1N4148W_SOD-123_SMD, F.Cu at (171.5, 134.3)
- added D34: 1N4148W, Diode:1N4148W_SOD-123_SMD, F.Cu at (189.0, 131.4)
- added D4: 1N4148W, Diode:1N4148W_SOD-123_SMD, F.Cu at (93.5, 79.0)
- added D5: 1N4148W, Diode:1N4148W_SOD-123_SMD, F.Cu at (111.5, 74.7)
- added D6: 1N4148W, Diode:1N4148W_SOD-123_SMD, F.Cu at (36.0, 111.5)
- added D7: 1N4148W, Diode:1N4148W_SOD-123_SMD, F.Cu at (54.4, 94.9)
- added D8: 1N4148W, Diode:1N4148W_SOD-123_SMD, F.Cu at (73.9, 83.3)
- added D9: 1N4148W, Diode:1N4148W_SOD-123_SMD, F.Cu at (93.5, 96.0)
- added H1: MountingHole, Mounting_Hole:3.2mm_M3_DIN965_Pad, F.Cu at (23.0, 64.0)
- added H2: MountingHole, Mounting_Hole:3.2mm_M3_DIN965_Pad, F.Cu at (141.0, 64.0)
- added H3: MountingHole, Mounting_Hole:3.2mm_M3_DIN965_Pad, F.Cu at (23.0, 146.5)
- added H4: MountingHole, Mounting_Hole:3.2mm_M3_DIN965_Pad, F.Cu at (141.0, 146.5)
- added H5: MountingHole, Mounting_Hole:3.2mm_M3_DIN965_Pad, F.Cu at (159.0, 64.0)
- added H6: MountingHole, Mounting_Hole:3.2mm_M3_DIN965_Pad, F.Cu at (277.0, 64.0)
- added H7: MountingHole, Mounting_Hole:3.2mm_M3_DIN965_Pad, F.Cu at (159.0, 146.5)
- added H8: MountingHole, Mounting_Hole:3.2mm_M3_DIN965_Pad, F.Cu at (277.0, 146.5)
- added SW1: PG1350, Kailh:PG1350_Choc_V1, F.Cu at (32.2, 99.7)
- added SW10: PG1350, Kailh:PG1350_Choc_V1, F.Cu at (111.5, 96.3)
- added SW11: PG1350, Kailh:PG1350_Choc_V1, F.Cu at (42.7, 132.0)
- added SW12: PG1350, Kailh:PG1350_Choc_V1, F.Cu at (57.8, 116.2)
- added SW13: PG1350, Kailh:PG1350_Choc_V1, F.Cu at (75.1, 104.9)
- added SW14: PG1350, Kailh:PG1350_Choc_V1, F.Cu at (93.5, 117.6)
- added SW15: PG1350, Kailh:PG1350_Choc_V1, F.Cu at (111.5, 113.3)
- added SW16: PG1350, Kailh:PG1350_Choc_V1, F.Cu at (110.1, 135.9)
- added SW17: PG1350, Kailh:PG1350_Choc_V1, F.Cu at (127.8, 138.7)
- added SW18: PG1350, Kailh:PG1350_Choc_V1, F.Cu at (188.5, 79.3)
- added SW19: PG1350, Kailh:PG1350_Choc_V1, F.Cu at (206.5, 83.6)
- added SW2: PG1350, Kailh:PG1350_Choc_V1, F.Cu at (52.5, 82.6)
- added SW20: PG1350, Kailh:PG1350_Choc_V1, F.Cu at (226.7, 71.0)
- added SW21: PG1350, Kailh:PG1350_Choc_V1, F.Cu at (247.6, 82.6)
- added SW22: PG1350, Kailh:PG1350_Choc_V1, F.Cu at (267.8, 99.7)
- added SW23: PG1350, Kailh:PG1350_Choc_V1, F.Cu at (188.5, 96.3)
- added SW24: PG1350, Kailh:PG1350_Choc_V1, F.Cu at (206.5, 100.6)
- added SW25: PG1350, Kailh:PG1350_Choc_V1, F.Cu at (225.8, 87.9)
- added SW26: PG1350, Kailh:PG1350_Choc_V1, F.Cu at (244.9, 99.4)
- added SW27: PG1350, Kailh:PG1350_Choc_V1, F.Cu at (262.6, 115.8)
- added SW28: PG1350, Kailh:PG1350_Choc_V1, F.Cu at (188.5, 113.3)
- added SW29: PG1350, Kailh:PG1350_Choc_V1, F.Cu at (206.5, 117.6)
- added SW3: PG1350, Kailh:PG1350_Choc_V1, F.Cu at (73.3, 71.0)
- added SW30: PG1350, Kailh:PG1350_Choc_V1, F.Cu at (224.9, 104.9)
- added SW31: PG1350, Kailh:PG1350_Choc_V1, F.Cu at (242.2, 116.2)
- added SW32: PG1350, Kailh:PG1350_Choc_V1, F.Cu at (257.3, 132.0)
- added SW33: PG1350, Kailh:PG1350_Choc_V1, F.Cu at (172.2, 138.7)
- added SW34: PG1350, Kailh:PG1350_Choc_V1, F.Cu at (189.9, 135.9)
- added SW4: PG1350, Kailh:PG1350_Choc_V1, F.Cu at (93.5, 83.6)
- added SW5: PG1350, Kailh:PG1350_Choc_V1, F.Cu at (111.5, 79.3)
- added SW6: PG1350, Kailh:PG1350_Choc_V1, F.Cu at (37.5, 115.8)
- added SW7: PG1350, Kailh:PG1350_Choc_V1, F.Cu at (55.1, 99.4)
- added SW8: PG1350, Kailh:PG1350_Choc_V1, F.Cu at (74.2, 87.9)
- added SW9: PG1350, Kailh:PG1350_Choc_V1, F.Cu at (93.5, 100.6)
- added U1: RP2040, Seed Studio:XIAO_RP2040_SMD, F.Cu at (29.5, 77.9)
- added U2: RP2040, Seed Studio:XIAO_RP2040_SMD, F.Cu at (270.5, 77.9)
Other:
- board outline added: 262 x 90.5 mm

Commit message: feat(pcb): implement keycap layout with stagger and splay for both sides
Parts:
- added H10: MountingHole, Mounting_Hole:3.2mm_M3_DIN965_Pad, F.Cu at (165.0, 130.5)
- added H11: MountingHole, Mounting_Hole:3.2mm_M3_DIN965_Pad, F.Cu at (210.4, 130.5)
- added H12: MountingHole, Mounting_Hole:3.2mm_M3_DIN965_Pad, F.Cu at (275.0, 130.5)
- added H9: MountingHole, Mounting_Hole:3.2mm_M3_DIN965_Pad, F.Cu at (165.0, 103.6)
- D1, D10, D11, D12, D13, D14, D15, D16, D17, D18, D19, D2, D20, D21, D22, D23, D24, D25, D26, D27, D28, D29, D3, D30, D31, D32, D33, D34, D4, D5, D6, D7, D8, D9: moved to B.Cu
- moved H6 156.6 mm to (135.0, 130.0)
- moved H3 119.9 mm to (134.8, 103.1), turned to 180 degrees
- moved H4 117.2 mm to (25.0, 130.0), turned to 180 degrees
- moved H7 100.2 mm to (165.0, 46.5), turned to 180 degrees
- moved H8 100.0 mm to (275.0, 46.5), turned to 180 degrees
- moved H5 95.8 mm to (89.6, 130.0)
- moved SW17 21.2 mm to (122.8, 118.1)
- moved D17 21.1 mm to (123.5, 113.7), turned to 171 degrees
- moved D33 20.8 mm to (176.5, 114.0), turned to -171 degrees
- moved SW33 20.8 mm to (177.2, 118.6)
- moved D16 20.6 mm to (103.6, 112.1), turned to 180 degrees
- moved SW16 20.4 mm to (103.6, 116.6), turned to 0 degrees
- moved D34 20.2 mm to (196.4, 112.6), turned to 180 degrees
- moved SW34 19.9 mm to (196.4, 117.1), turned to 0 degrees
- moved H2 19.0 mm to (135.0, 46.0)
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Connections:
- U1 pad 13: unconnected-(U1-GND-Pad13) -> GND_L
Routing:
- net ROW0_R: track 0.00 -> 22.2 mm
- net ROW1_R: track 0.13 -> 16.8 mm
- net ROW2_R: track 0.00 -> 14.0 mm
- net ROW3_R: track 0.00 -> 11.4 mm
- net Net-(D19-A): track 0.00 -> 9.70 mm
- net Net-(D24-A): track 0.00 -> 9.70 mm
- net Net-(D4-A): track 0.00 -> 9.70 mm
- net Net-(D34-A): track 0.00 -> 9.70 mm
- net Net-(D18-A): track 0.00 -> 9.70 mm
- net Net-(D29-A): track 0.00 -> 9.70 mm
- net Net-(D10-A): track 0.00 -> 9.70 mm
- net Net-(D16-A): track 0.00 -> 9.70 mm
- net Net-(D14-A): track 0.00 -> 9.70 mm
- net Net-(D5-A): track 0.00 -> 9.70 mm
- net Net-(D9-A): track 0.00 -> 9.70 mm
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Other:
- board size 262 x 90.5 mm -> 257 x 91.5 mm
